Commit message: 增加irmv2

File: resources/robots/irmv_v2/irmv_v2_0319.urdf (robot description, URDF)
Before this commit: robot irmv_v2_0319, 14 links, 13 joints
Links:
- link Link_ankle_l_pitch: geometry collision mesh filename=./meshes/Link_ankle_l_pitch.STL; visual mesh filename=./meshes/Link_ankle_l_pitch.STL
- link Link_ankle_l_roll: mass 0.22291 -> 0.32291; geometry collision mesh filename=./meshes/Link_ankle_l_roll.STL; visual mesh filename=./meshes/Link_ankle_l_roll.STL
- link Link_ankle_r_pitch: geometry collision mesh filename=./meshes/Link_ankle_r_pitch.STL; visual mesh filename=./meshes/Link_ankle_r_pitch.STL
- link Link_ankle_r_roll: mass 0.22291 -> 0.32291; geometry collision mesh filename=./meshes/Link_ankle_r_roll.STL; visual mesh filename=./meshes/Link_ankle_r_roll.STL
- link Link_base: geometry collision mesh filename=./meshes/Link_base.STL; visual mesh filename=./meshes/Link_base.STL
- link Link_body: geometry collision mesh filename=./meshes/Link_body.STL; visual mesh filename=./meshes/Link_body.STL
- link Link_hip_l_pitch: geometry collision mesh filename=./meshes/Link_hip_l_pitch.STL; visual mesh filename=./meshes/Link_hip_l_pitch.STL
- link Link_hip_l_roll: geometry collision mesh filename=./meshes/Link_hip_l_roll.STL; visual mesh filename=./meshes/Link_hip_l_roll.STL
- link Link_hip_l_yaw: geometry collision mesh filename=./meshes/Link_hip_l_yaw.STL; visual mesh filename=./meshes/Link_hip_l_yaw.STL
- link Link_hip_r_pitch: geometry collision mesh filename=./meshes/Link_hip_r_pitch.STL; visual mesh filename=./meshes/Link_hip_r_pitch.STL
- link Link_hip_r_roll: geometry collision mesh filename=./meshes/Link_hip_r_roll.STL; visual mesh filename=./meshes/Link_hip_r_roll.STL
- link Link_hip_r_yaw: geometry collision mesh filename=./meshes/Link_hip_r_yaw.STL; visual mesh filename=./meshes/Link_hip_r_yaw.STL
- link Link_knee_l_pitch: geometry collision cylinder length=0.02 radius=0.03; visual mesh filename=./meshes/Link_knee_l_pitch.STL
- link Link_knee_r_pitch: geometry collision cylinder length=0.02 radius=0.03; visual mesh filename=./meshes/Link_knee_r_pitch.STL
Joints:
- joint Joint_ankle_l_pitch: axis 0 -1 0 -> 0 1 0; limit lower=0 upper=0 effort=0 velocity=0 -> lower=-0.7854 upper=0.8727 effort=30 velocity=6
- joint Joint_ankle_r_pitch: axis 0 -1 0 -> 0 1 0; limit lower=0 upper=0 effort=0 velocity=0 -> lower=-0.7854 upper=0.8727 effort=30 velocity=6
- joint Joint_hip_l_pitch: axis 0 -1 0 -> 0 1 0; limit lower=0 upper=0 effort=0 velocity=0 -> lower=-2.2689 upper=0.9948 effort=40 velocity=12
- joint Joint_hip_l_roll: limit lower=-1.5708 upper=1.5708 effort=0 velocity=0 -> lower=-1.5708 upper=1.5708 effort=35 velocity=3
- joint Joint_hip_l_yaw: limit lower=-1.5708 upper=1.5708 effort=0 velocity=0 -> lower=-1.5708 upper=1.5708 effort=35 velocity=3
- joint Joint_hip_r_pitch: axis 0 -1 0 -> 0 1 0; limit lower=0 upper=0 effort=0 velocity=0 -> lower=-2.2689 upper=0.9948 effort=40 velocity=12
- joint Joint_hip_r_roll: limit lower=-1.5708 upper=1.5708 effort=0 velocity=0 -> lower=-1.5708 upper=1.5708 effort=35 velocity=3
- joint Joint_hip_r_yaw: limit lower=-1.5708 upper=1.5708 effort=0 velocity=0 -> lower=-1.5708 upper=1.5708 effort=35 velocity=3
- joint Joint_knee_l_pitch: axis 0 -1 0 -> 0 1 0; limit lower=0 upper=0 effort=0 velocity=0 -> lower=0 upper=2.0944 effort=40 velocity=12
- joint Joint_knee_r_pitch: axis 0 -1 0 -> 0 1 0; limit lower=0 upper=0 effort=0 velocity=0 -> lower=0 upper=2.0944 effort=40 velocity=12
